Commit message: renders

File: quad_simulator/vision60_description/urdf/vision60.urdf (robot description, URDF)
Before this commit: robot ngr, 17 links, 16 joints
Links:
- link body: mass 12 -> 25; geometry collision box size=0.83 0.25 0.19; visual mesh filename=package://vision60_description/meshes/v5_body_decimated.stl scale=1.0 1.0 1.0
- link hip0: mass 2.75 -> 1.975; geometry collision box size=0.15 0.09 0.15; visual mesh filename=package://vision60_description/meshes/v5_pod_decimated.stl scale=1.0 1.0 1.0
- link hip1: mass 2.75 -> 1.975; geometry collision box size=0.15 0.09 0.15; visual mesh filename=package://vision60_description/meshes/v5_pod_decimated.stl scale=1.0 1.0 1.0
- link hip2: mass 2.75 -> 1.975; geometry collision box size=0.15 0.09 0.15; visual mesh filename=package://vision60_description/meshes/v5_pod_decimated.stl scale=1.0 1.0 1.0
- link hip3: mass 2.75 -> 1.975; geometry collision box size=0.15 0.09 0.15; visual mesh filename=package://vision60_description/meshes/v5_pod_decimated.stl scale=1.0 1.0 1.0
- link lower0: mass 0.2 -> 0.375; geometry collision cylinder length=0.3407 radius=0.02; visual mesh filename=package://vision60_description/meshes/v5_lower_decimated.stl scale=1.0 1.0 1.0
- link lower1: mass 0.2 -> 0.375; geometry collision cylinder length=0.3407 radius=0.02; visual mesh filename=package://vision60_description/meshes/v5_lower_decimated.stl scale=1.0 1.0 1.0
- link lower2: mass 0.2 -> 0.375; geometry collision cylinder length=0.3407 radius=0.02; visual mesh filename=package://vision60_description/meshes/v5_lower_decimated.stl scale=1.0 1.0 1.0
- link lower3: mass 0.2 -> 0.375; geometry collision cylinder length=0.3407 radius=0.02; visual mesh filename=package://vision60_description/meshes/v5_lower_decimated.stl scale=1.0 1.0 1.0
- link toe0: geometry collision sphere radius=0.035; visual sphere radius=0.035
- link toe1: geometry collision sphere radius=0.035; visual sphere radius=0.035
- link toe2: geometry collision sphere radius=0.035; visual sphere radius=0.035
- link toe3: geometry collision sphere radius=0.035; visual sphere radius=0.035
- link upper0: mass 0.625 -> 2.525; geometry collision box size=0.34 0.055 0.075; visual mesh filename=package://vision60_description/meshes/v5_left_upper_decimat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 scale=1.0 1.0 1.0
- link upper1: mass 0.625 -> 2.525; geometry collision box size=0.34 0.055 0.075; visual mesh filename=package://vision60_description/meshes/v5_left_upper_decimat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 scale=1.0 1.0 1.0
- link upper2: mass 0.625 -> 2.525; geometry collision box size=0.34 0.055 0.075; visual mesh filename=package://vision60_description/meshes/v5_right_upper_decima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 scale=1.0 1.0 1.0
- link upper3: mass 0.625 -> 2.525; geometry collision box size=0.34 0.055 0.075; visual mesh filename=package://vision60_description/meshes/v5_right_upper_decima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 scale=1.0 1.0 1.0
Joints:
- joint 0: limit lower=-3.14159265359 upper=3.14159265359 effort=87.5 velocity=30 -> lower=-6.28 upper=6.28 effort=87.5 velocity=30; origin xyz=0 0.068 0 -> xyz=0 0.1221 0
- joint 1: limit lower=0 upper=3.14159265359 effort=87.5 velocity=30 -> lower=0.3 upper=2.6 effort=87.5 velocity=30; origin xyz=-0.25 0 0 -> xyz=-0.34 0 0
- joint 10: origin xyz=0.325 -0.1575 0 -> xyz=0.3075 -0.1 0
- joint 11: origin xyz=-0.325 -0.1575 0 -> xyz=-0.3075 -0.1 0
- joint 2: limit lower=-3.14159265359 upper=3.14159265359 effort=87.5 velocity=30 -> lower=-3.8 upper=2.27 effort=87.5 velocity=30; origin xyz=0 0.068 0 -> xyz=0 0.1221 0
- joint 3: limit lower=0 upper=3.14159265359 effort=87.5 velocity=30 -> lower=0.3 upper=2.6 effort=87.5 velocity=30; origin xyz=-0.25 0 0 -> xyz=-0.34 0 0
- joint 4: limit lower=-3.14159265359 upper=3.14159265359 effort=87.5 velocity=30 -> lower=-6.28 upper=6.28 effort=87.5 velocity=30; origin xyz=0 -0.068 0 -> xyz=0 -0.1221 0
- joint 5: limit lower=0 upper=3.14159265359 effort=87.5 velocity=30 -> lower=0.3 upper=2.6 effort=87.5 velocity=30; origin xyz=-0.25 0 0 -> xyz=-0.34 0 0
- joint 6: limit lower=-3.14159265359 upper=3.14159265359 effort=87.5 velocity=30 -> lower=-3.8 upper=2.27 effort=87.5 velocity=30; origin xyz=0 -0.068 0 -> xyz=0 -0.1221 0
- joint 7: limit lower=0 upper=3.14159265359 effort=87.5 velocity=30 -> lower=0.3 upper=2.6 effort=87.5 velocity=30; origin xyz=-0.25 0 0 -> xyz=-0.34 0 0
- joint 8: origin xyz=0.325 0.1575 0 -> xyz=0.3075 0.1 0
- joint 9: origin xyz=-0.325 0.1575 0 -> xyz=-0.3075 0.1 0
- joint jtoe0: origin xyz=0.28 0 -0.0461 -> xyz=0.3407 0 0
- joint jtoe1: origin xyz=0.28 0 -0.0461 -> xyz=0.3407 0 0
- joint jtoe2: origin xyz=0.28 0 -0.0461 -> xyz=0.3407 0 0
- joint jtoe3: origin xyz=0.28 0 -0.0461 -> xyz=0.3407 0 0
